File: stez80/cpu.kicad_sch (KiCad schematic)
At the start: 10 parts, among them J1 Conn_01x32_Pin, U1 74HC14, U2 Z80CPU, U3 AS6C1008-xxP, U4 27C512

Commit message: pcb layout
Parts:
- renumbered C2 to C1, C1 to C2
Connections:
- net ~{NMI} is gone; now on an unnamed net: U2.17 (~{NMI})
- net AddressBus0: now also J1.17 (Pin_17); no longer J1.24 (Pin_24)
- net AddressBus1: now also J1.18 (Pin_18); no longer J1.23 (Pin_23)
- net AddressBus10: now also J1.27 (Pin_27); no longer J1.14 (Pin_14)
- net AddressBus11: now also J1.28 (Pin_28); no longer J1.13 (Pin_13)
- net AddressBus12: now also J1.29 (Pin_29); no longer J1.12 (Pin_12)
- net AddressBus13: now also J1.30 (Pin_30); no longer J1.11 (Pin_11)
- net AddressBus14: now also J1.31 (Pin_31); no longer J1.10 (Pin_10)
- net AddressBus15: now also J1.32 (Pin_32); no longer J1.9 (Pin_9)
- net AddressBus2: now also J1.19 (Pin_19); no longer J1.22 (Pin_22)
- net AddressBus3: now also J1.20 (Pin_20); no longer J1.21 (Pin_21)
- net AddressBus4: now also J1.21 (Pin_21); no longer J1.20 (Pin_20)
- net AddressBus5: now also J1.22 (Pin_22); no longer J1.19 (Pin_19)
- net AddressBus6: now also J1.23 (Pin_23); no longer J1.18 (Pin_18)
- net AddressBus7: now also J1.24 (Pin_24); no longer J1.17 (Pin_17)
- net AddressBus8: now also J1.25 (Pin_25); no longer J1.16 (Pin_16)
- net AddressBus9: now also J1.26 (Pin_26); no longer J1.15 (Pin_15)
- net Databus0: now also J1.9 (Pin_9); no longer J1.32 (Pin_32)
- net Databus1: now also J1.10 (Pin_10); no longer J1.31 (Pin_31)
- net Databus2: now also J1.11 (Pin_11); no longer J1.30 (Pin_30)
- net Databus3: now also J1.12 (Pin_12); no longer J1.29 (Pin_29)
- net Databus4: now also J1.13 (Pin_13); no longer J1.28 (Pin_28)
- net Databus5: now also J1.14 (Pin_14); no longer J1.27 (Pin_27)
- net Databus6: now also J1.15 (Pin_15); no longer J1.26 (Pin_26)
- net Databus7: now also J1.16 (Pin_16); no longer J1.25 (Pin_25)

Commit message: review wip
Parts:
- U3: value AS6C1008-xxP -> AS6C1008-55PCN; footprint Package_DIP:DIP-32_W15.24mm -> Package_DIP:DIP-32_W15.24mm_LongPads
- U4: footprint Package_DIP:DIP-28_W15.24mm -> Package_DIP:DIP-28_W15.24mm_LongPads
Changed lines of the file:
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@@
 	(title_block
 		(title "Ste z80 board")
+		(date "2025-05-11")
 		(rev "V0.1")
 	)
-	(text_box "74hc14 unsed/power"
+	(text_box "74hc14 unused/power"
 		(exclude_from_sim no)
 		(at 16.51 135.89 0)
@@
 			)
 		)
-		(property "Value" "AS6C1008-xxP"
+		(property "Value" "AS6C1008-55PCN"
 			(at 172.3233 45.72 0)
 			(effects
@@
 			)
 		)
-		(property "Footprint" "Package_DIP:DIP-32_W15.24mm"
+		(property "Footprint" "Package_DIP:DIP-32_W15.24mm_LongPads"
 			(at 170.18 71.12 0)
 			(effects
@@
 			)
 		)
-		(property "Datasheet" "https://www.alliancememory.com/wp-content/uploads/pdf/AS6C1008_Mar_2023V1.2.pdf"
+		(property "Datasheet" "kicad-embed://AS6C1008.PDF"
 			(at 170.18 71.12 0)
 			(effects
@@
 			)
 		)
-		(property "Datasheet" "www.zilog.com/manage_directlink.php?filepath=docs/z80/um0080"
+		(property "Datasheet" "kicad-embed://Z8400.PDF"
 			(at 59.69 71.12 0)
 			(effects
@@
 			)
 		)
-		(property "Footprint" "Package_DIP:DIP-28_W15.24mm"
+		(property "Footprint" "Package_DIP:DIP-28_W15.24mm_LongPads"
 			(at 243.84 76.2 0)
 			(effects

Commit message: continue review
Parts:
- renumbered C2 to C1, C1 to C2
Changed lines of the file:
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@@
 		(dnp no)
 		(fields_autoplaced yes)
-		(property "Reference" "C1"
+		(property "Reference" "C2"
 			(at 109.22 148.5899 0)
 			(effects
@@
 			(project "stez80"
 				(path "/8f25e73c-50ea-4100-9671-d49097d9068a/a5ee72ab-b6ae-4be4-95d4-715b05ad0242"
-					(reference "C1")
+					(reference "C2")
 					(unit 1)
 				)
@@
 		(dnp no)
 		(fields_autoplaced yes)
-		(property "Reference" "C2"
+		(property "Reference" "C1"
 			(at 52.07 38.0999 0)
 			(effects
@@
 			(project "stez80"
 				(path "/8f25e73c-50ea-4100-9671-d49097d9068a/a5ee72ab-b6ae-4be4-95d4-715b05ad0242"
-					(reference "C2")
+					(reference "C1")
 					(unit 1)
 				)
