File: stez80/stez80.kicad_pcb (KiCad board)
At the start: 4 copper layers, 100 x 100 mm, 38 parts, among them J1 Conn_01x32_Pin, J2 Barrel_Jack, J3 DE9_Socket, SW1 SW_Push, U1 74HC14, U2 Z80CPU, U3 AS6C1008-xxP, U4 27C512, U5 ATmega16A-P, U6 Z80_SIO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

Commit message: pcb layout
Parts:
- J2: footprint Connector_BarrelJack:BarrelJack_CUI_PJ-063AH_Horizontal_CircularHoles -> Connector_BarrelJack:BarrelJack_CUI_PJ-063AH_Horizontal
- J3: footprint Connector_Dsub:DSUB-9_Socket_Horizontal_P2.77x2.84mm_EdgePinOffset4.94mm_Housed_MountingHolesOffset4.94mm -> Connector_Dsub:DSUB-9_Socket_Horizontal_P2.77x2.84mm_EdgePinOffset7.70mm_Housed_MountingHolesOffset9.12mm
- moved C9 83.2 mm to (80.6, 104.4)
- moved C1 78.4 mm to (72.3, 102.6)
- moved U6 77.0 mm to (66.4, 99.1), turned to 90 degrees
- moved C2 74.5 mm to (42.5, 26.5)
- moved U4 69.1 mm to (81.0, 30.0)
- moved JP2 59.6 mm to (104.4, 26.0), turned to 90 degrees
- moved JP4 48.3 mm to (79.0, 26.0), turned to 90 degrees
- moved C7 39.6 mm to (42.0, 105.0)
- moved U1 37.7 mm to (62.3, 121.0), turned to 90 degrees
- moved C12 30.6 mm to (65.5, 108.5)
- moved R3 27.1 mm to (80.0, 109.5)
- moved R2 24.6 mm to (57.5, 112.1), turned to -90 degrees
- moved C6 24.0 mm to (49.5, 107.0), turned to 90 degrees
- moved D1 23.2 mm to (58.1, 90.5)
- moved JP3 22.8 mm to (83.0, 68.7)
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- renumbered JP5 to JP3, JP3 to JP4, JP4 to JP5
Connections:
- J1 pad 10: AddressBus14 -> Databus1
- J1 pad 11: AddressBus13 -> Databus2
- J1 pad 12: AddressBus12 -> Databus3
- J1 pad 13: AddressBus11 -> Databus4
- J1 pad 14: AddressBus10 -> Databus5
- J1 pad 15: AddressBus9 -> Databus6
- J1 pad 16: AddressBus8 -> Databus7
- J1 pad 17: AddressBus7 -> AddressBus0
- J1 pad 18: AddressBus6 -> AddressBus1
- J1 pad 19: AddressBus5 -> AddressBus2
- J1 pad 20: AddressBus4 -> AddressBus3
- J1 pad 21: AddressBus3 -> AddressBus4
- J1 pad 22: AddressBus2 -> AddressBus5
- J1 pad 23: AddressBus1 -> AddressBus6
- J1 pad 24: AddressBus0 -> AddressBus7
- J1 pad 25: Databus7 -> AddressBus8
- J1 pad 26: Databus6 -> AddressBus9
- J1 pad 27: Databus5 -> AddressBus10
- J1 pad 28: Databus4 -> AddressBus11
- J1 pad 29: Databus3 -> AddressBus12
- J1 pad 30: Databus2 -> AddressBus13
- J1 pad 31: Databus1 -> AddressBus14
- J1 pad 32: Databus0 -> AddressBus15
- J1 pad 9: AddressBus15 -> Databus0
- U2 pad 17: ~{NMI} -> Net-(U2-~{BUSRQ})
- U5 pad 33: AddressBus7 -> AddressBus0
- U5 pad 34: AddressBus6 -> AddressBus1
- U5 pad 35: AddressBus5 -> AddressBus2
- U5 pad 36: AddressBus4 -> AddressBus3
- U5 pad 37: AddressBus3 -> AddressBus4
- U5 pad 38: AddressBus2 -> AddressBus5
- U5 pad 39: AddressBus1 -> AddressBus6
- U5 pad 40: AddressBus0 -> AddressBus7
Routing:
- net ~{RESET}: track 0.00 -> 201.9 mm, vias 0 -> 9
- net AddressBus0: track 0.00 -> 198.4 mm, vias 0 -> 11
- net Databus3: track 0.00 -> 185.0 mm, vias 0 -> 10
- net Databus7: track 0.00 -> 174.4 mm, vias 0 -> 8
- net Databus5: track 0.00 -> 171.3 mm, vias 0 -> 9
- net ~{WR}: track 0.00 -> 170.4 mm, vias 0 -> 6
- net Databus1: track 0.00 -> 169.3 mm, vias 0 -> 9
- net ~{RD}: track 0.00 -> 164.8 mm, vias 0 -> 6
- net Databus4: track 0.00 -> 164.5 mm, vias 0 -> 9
- net ~{INT}: track 0.00 -> 162.6 mm, vias 0 -> 9
- net Databus0: track 0.00 -> 153.7 mm, vias 0 -> 8
- net AddressBus1: track 0.00 -> 153.1 mm, vias 0 -> 8
- net Databus2: track 0.00 -> 151.6 mm, vias 0 -> 7
- net Databus6: track 0.00 -> 149.7 mm, vias 0 -> 6
- net AddressBus2: track 0.00 -> 144.5 mm, vias 0 -> 8
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
Commit message: review wip
Parts:
- U3: value AS6C1008-xxP -> AS6C1008-55PCN; footprint Package_DIP:DIP-32_W15.24mm -> Package_DIP:DIP-32_W15.24mm_LongPads
- U4: footprint Package_DIP:DIP-28_W15.24mm -> Package_DIP:DIP-28_W15.24mm_LongPads
- U5: footprint Package_DIP:DIP-40_W15.24mm -> Package_DIP:DIP-40_W15.24mm_LongPads
Routing:
- net AddressBus1: track 153.1 -> 143.1 mm
- net AddressBus0: track 198.4 -> 188.4 mm
- net AddressBus2: track 144.5 -> 134.7 mm
- net AddressBus3: track 143.3 -> 134.2 mm
- net AddressBus4: track 140.1 -> 132.4 mm
- net AddressBus5: track 137.5 -> 130.4 mm
- net AddressBus6: track 122.6 -> 115.6 mm
- net AddressBus9: track 130.2 -> 125.7 mm
- net AddressBus10: track 139.5 -> 138.5 mm
- net AddressBus11: track 139.2 -> 138.4 mm
- net MA14: track 60.5 -> 61.1 mm
- net AddressBus8: track 120.4 -> 120.9 mm
- net Databus5: track 171.3 -> 171.8 mm

Commit message: continue review
Parts:
- added C16: 100nF, Capacitor_THT:C_Rect_L7.0mm_W2.0mm_P5.00mm, F.Cu at (119.5, 63.7)
- J2: footprint Connector_BarrelJack:BarrelJack_CUI_PJ-063AH_Horizontal -> Connector_BarrelJack:BarrelJack_GCT_DCJ200-10-A_Horizontal
- U7: footprint Package_DIP:DIP-16_W7.62mm -> Package_DIP:DIP-16_W7.62mm_LongPads
- moved C2 88.7 mm to (70.2, 110.8)
- moved C1 57.3 mm to (39.9, 55.3), turned to 90 degrees
- moved C3 12.6 mm to (75.6, 26.9), turned to 180 degrees
- moved C11 9.37 mm to (133.0, 89.1), turned to -90 degrees
- moved C9 6.32 mm to (86.5, 102.2), turned to 180 degrees
- moved J2 3.92 mm to (46.3, 109.6)
- moved C6 1.97 mm to (49.6, 105.0)
- moved C7 1.41 mm to (40.6, 105.0)
Routing:
- net Net-(D1-A): track 25.5 -> 21.8 mm
- net AddressBus1: track 143.1 -> 139.4 mm
- net AddressBus0: track 188.4 -> 185.3 mm
- net MA14: track 61.1 -> 62.9 mm
- net MA15: track 10.3 -> 8.67 mm, vias 2 -> 0
- net Databus6: track 150.1 -> 151.5 mm
- net ~{M1}: track 143.0 -> 144.0 mm
- net AddressBus2: track 134.7 -> 135.7 mm
- net Databus7: track 174.2 -> 174.9 mm

Commit message: v0.1
Parts:
- C10, C13, C14, C15: value 100nF -> 1uF
- SW1: footprint Button_Switch_THT:SW_PUSH-12mm -> Button_Switch_THT:SW_PUSH_6mm_H7.3mm
- moved C4 71.3 mm to (93.1, 26.0), turned to 180 degrees
- moved C5 40.9 mm to (96.1, 66.9), turned to -90 degrees
- moved C8 7.12 mm to (120.8, 47.8), turned to 0 degrees
- moved JP5 5.80 mm to (128.1, 43.5)
- moved R3 0.71 mm to (80.7, 109.7)
- moved SW1 0.30 mm to (83.5, 113.3)
Routing:
- net ATMEGA_CLK: track 33.6 -> 39.8 mm
- net Net-(R3-Pad1): track 35.1 -> 30.3 mm
- net Net-(JP5-A): track 7.23 -> 8.38 mm
Other:
- board text added: "steZ80 v0.1 5.2025 Stefan Aeschbacher"
- board text removed: "steZ80 (c) 2025 Stefan Aeschbacher"
