File: stez80/support.kicad_sch (KiCad schematic)
At the start: 29 parts, among them J2 Barrel_Jack, J3 DE9_Socket, SW1 SW_Push, U1 74HC14, U5 ATmega16A-P, U6 Z80_SIO, U7 MAX232, Y1 CXO_DIP8

Commit message: pcb layout
Parts:
- J2: footprint Connector_BarrelJack:BarrelJack_CUI_PJ-063AH_Horizontal_CircularHoles -> Connector_BarrelJack:BarrelJack_CUI_PJ-063AH_Horizontal
- J3: footprint Connector_Dsub:DSUB-9_Socket_Horizontal_P2.77x2.84mm_EdgePinOffset4.94mm_Housed_MountingHolesOffset4.94mm -> Connector_Dsub:DSUB-9_Socket_Horizontal_P2.77x2.84mm_EdgePinOffset7.70mm_Housed_MountingHolesOffset9.12mm
Connections:
- net AddressBus0: now also U5.33 (PA7); no longer U5.40 (PA0)
- net AddressBus1: now also U5.34 (PA6); no longer U5.39 (PA1)
- net AddressBus2: now also U5.35 (PA5); no longer U5.38 (PA2)
- net AddressBus3: now also U5.36 (PA4); no longer U5.37 (PA3)
- net AddressBus4: now also U5.37 (PA3); no longer U5.36 (PA4)
- net AddressBus5: now also U5.38 (PA2); no longer U5.35 (PA5)
- net AddressBus6: now also U5.39 (PA1); no longer U5.34 (PA6)
- net AddressBus7: now also U5.40 (PA0); no longer U5.33 (PA7)
Changed lines of the file:
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@@
 		)
 	)
-	(label "AddressBus4"
+	(label "AddressBus3"
 		(at 92.71 62.23 180)
 		(effects
@@
 		)
 	)
-	(label "AddressBus5"
+	(label "AddressBus2"
 		(at 92.71 64.77 180)
 		(effects
@@
 		)
 	)
-	(label "AddressBus7"
+	(label "AddressBus0"
 		(at 92.71 69.85 180)
 		(effects
@@
 		)
 	)
-	(label "AddressBus6"
+	(label "AddressBus1"
 		(at 92.71 67.31 180)
 		(effects
@@
 		)
 	)
-	(label "AddressBus0"
+	(label "AddressBus7"
 		(at 92.71 52.07 180)
 		(effects
@@
 		)
 	)
-	(label "AddressBus2"
+	(label "AddressBus5"
 		(at 92.71 57.15 180)
 		(effects
@@
 		)
 	)
-	(label "AddressBus3"
+	(label "AddressBus4"
 		(at 92.71 59.69 180)
 		(effects
@@
 		)
 	)
-	(label "AddressBus1"
+	(label "AddressBus6"
 		(at 92.71 54.61 180)
 		(effects
@@
 			)
 		)
-		(property "Footprint" "Connector_BarrelJack:BarrelJack_CUI_PJ-063AH_Horizontal_CircularHoles"
+		(property "Footprint" "Connector_BarrelJack:BarrelJack_CUI_PJ-063AH_Horizontal"
 			(at 26.67 177.546 0)
 			(effects
@@
 			)
 		)
-		(property "Footprint" "Connector_Dsub:DSUB-9_Socket_Horizontal_P2.77x2.84mm_EdgePinOffset4.94mm_Housed_MountingHolesOffset4.94mm"
+		(property "Footprint" "Connector_Dsub:DSUB-9_Socket_Horizontal_P2.77x2.84mm_EdgePinOffset7.70mm_Housed_MountingHolesOffset9.12mm"
 			(at 276.86 101.6 0)
 			(effects

Commit message: review wip
Parts:
- U5: footprint Package_DIP:DIP-40_W15.24mm -> Package_DIP:DIP-40_W15.24mm_LongPads
- U7: footprint Package_DIP:DIP-16_W7.62mm -> Package_DIP:DIP-16_W7.62mm_LongPads
Changed lines of the file:
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@@
 	(title_block
 		(title "Ste z80 board")
+		(date "2025-05-11")
 		(rev "V0.1")
 	)
@@
 			)
 		)
-		(property "Footprint" "Package_DIP:DIP-40_W15.24mm"
+		(property "Footprint" "Package_DIP:DIP-40_W15.24mm_LongPads"
 			(at 53.34 95.25 0)
 			(effects
@@
 			)
 		)
-		(property "Footprint" "Package_DIP:DIP-16_W7.62mm"
+		(property "Footprint" "Package_DIP:DIP-16_W7.62mm_LongPads"
 			(at 238.76 96.52 0)
 			(effects

Commit message: continue review
Parts:
- removed C12, C7: 1uF, Capacitor_THT:CP_Radial_D5.0mm_P2.50mm, symbol Device:C
- added C12, C7: 1uF, Capacitor_THT:CP_Radial_D5.0mm_P2.50mm, symbol Device:C_Polarized
- added C16: 100nF, Capacitor_THT:C_Rect_L7.0mm_W2.0mm_P5.00mm, symbol Device:C
- C10, C13, C14, C15: value 100nF -> 1uF
- J2: footprint Connector_BarrelJack:BarrelJack_CUI_PJ-063AH_Horizontal -> Connector_BarrelJack:BarrelJack_GCT_DCJ200-10-A_Horizontal
Connections:
- net GND: now also C12.2, C16.2, C7.2
- net VCC: now also C16.1, C7.1
- net at R4.2, U1.1: now also C12.1

Commit message: v0.1
Parts:
- SW1: footprint Button_Switch_THT:SW_PUSH-12mm -> Button_Switch_THT:SW_PUSH_6mm_H7.3mm
Changed lines of the file:
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@@
 		(exclude_from_sim no)
 		(at 17.78 16.51 0)
-		(size 111.76 139.7)
+		(size -111.76 139.7)
 		(margins 0.9525 0.9525 0.9525 0.9525)
 		(stroke
@@
 				(size 1.27 1.27)
 			)
-			(justify left top)
+			(justify right top)
 		)
 	)
@@
 			)
 		)
-		(property "Footprint" "Button_Switch_THT:SW_PUSH-12mm"
+		(property "Footprint" "Button_Switch_THT:SW_PUSH_6mm_H7.3mm"
 			(at 204.47 147.32 0)
 			(effects
